File: STM32Inverter.kicad_sch (KiCad schematic)
At the start: 63 parts, among them J1 STLINK, J2 RESOLVER, J3 MAIN POWER, J4 Power, J5 UART, J6 INTERFACE, J7 CURRENT SENSE, J8 DRIVER BOARD, U1 STM32F303VCTx, U4 74HCT00, U7 MCP2551-I-SN, Y3 CSTNE8M00GH5C000R0

Commit message: Schematic cleanup. Pinout changed
Parts:
- removed F4: 2A, symbol Device:Fuse
- removed J6: INTERFACE, Connector_IDC:IDC-Header_2x08_P2.54mm_Vertical, symbol Connector_Generic:Conn_02x08_Odd_Even
- added C17, C29, C30: 100n, Capacitor_SMD:C_0603_1608Metric_Pad1.08x0.95mm_HandSolder, symbol Device:C
- added D9: PESD3V3L5UY, Package_TO_SOT_SMD:SOT-363_SC-70-6, symbol Power_Protection:PESD3V3L5UY
- added F4: 350mA, Fuse:Fuse_0805_2012Metric, symbol Device:Polyfuse
- added F5: 2A, Fuse:Fuse_0805_2012Metric, symbol Device:Polyfuse
- added H1: M4, MountingHole:MountingHole_4.3mm_M4_ISO7380_Pad, symbol Mechanical:MountingHole_Pad
- added H2, H3, H4: MountingHole_Pad, MountingHole:MountingHole_4.3mm_M4_ISO7380_Pad, symbol Mechanical:MountingHole_Pad
- added J9: INTERFACE, Connector_IDC:IDC-Header_2x10_P2.54mm_Vertical, symbol Connector_Generic:Conn_02x10_Odd_Even
- added R33, R37, R38, R39, R40, R42, R44: 10k, Resistor_SMD:R_0603_1608Metric_Pad0.98x0.95mm_HandSolder, symbol Device:R
- added R41, R43, R45: 2.2k, Resistor_SMD:R_0603_1608Metric_Pad0.98x0.95mm_HandSolder, symbol Device:R
- added U10: ULN2002, Package_SO:SOP-16_3.9x9.9mm_P1.27mm, symbol Transistor_Array:ULN2002
- J1: footprint (none) -> Connector_PinHeader_2.54mm:PinHeader_1x04_P2.54mm_Vertical
- J2: footprint Connector_IDC:IDC-Header_2x06_P2.54mm_Horizontal -> Connector_IDC:IDC-Header_2x06_P2.54mm_Vertical
- J3: footprint (none) -> Connector_JST:JST_XH_B2B-XH-AM_1x02_P2.50mm_Vertical
- J4: footprint Connector_IDC:IDC-Header_2x03_P2.54mm_Horizontal -> Connector_PinHeader_2.54mm:PinHeader_1x06_P2.54mm_Vertical
- J8: footprint Connector_IDC:IDC-Header_2x10_P2.54mm_Horizontal -> Connector_IDC:IDC-Header_2x10_P2.54mm_Vertical
- R18: value R -> 470
Connections:
- net +12_EXT: now also F5.2, J9.1 (Pin_1), J9.3 (Pin_3)
- net CAN_H: now also J9.2 (Pin_2)
- net CAN_L: now also J9.4 (Pin_4)
- net GND: now also C17.2, C29.2, C30.2, D9.2 (A), H1.1, H2.1, H3.1, H4.1, J9.10 (Pin_10), J9.5 (Pin_5), J9.7 (Pin_7), R37.2, R39.2, R41.2, R43.2, R45.2, U10.8 (GND)
- net SWCLK: now also J9.14 (Pin_14); no longer J1.3 (Pin_3)
- net SWDIO: now also J9.12 (Pin_12); no longer J1.2 (Pin_2)
- net +12_UNSTABILIZED: now reaches D4.1 (K), J3.1 (Pin_1), R29.1
- net +12_UNSTABILIZED: now also F5.1, U10.9 (COM)
- net at F3.2: now also J9.16 (Pin_16)
- net +12V: no longer names the net of J4.6 (Pin_6)
- net +12V: now also F4.2; no longer C21.1
- new net: J9.19 (Pin_19), R44.1
- new net: J9.20 (Pin_20), R42.1
- new net: J9.8 (Pin_8), R33.1
- new net: J9.6 (Pin_6), R38.1
- new net: J9.18 (Pin_18), R40.1
- new net +15V: C21.1, F4.1
- new net ACC_INPUT_A_3V3: D9.1 (K1), R33.2, R37.1
- new net ACC_INPUT_B_3V3: D9.3 (K2), R38.2, R39.1
- new net AUX_IN: C30.1, D9.6 (K5), R44.2, R45.1
- new net BRK_IN: C29.1, D9.5 (K4), R40.2, R41.1
- new net FAN_OUT: U10.2 (I2)
- new net FAN_OUT_OD: J9.11 (Pin_11), U10.15 (O2)
- new net KEY_IN: C17.1, D9.4 (K3), R42.2, R43.1
- new net MAIN_OUT: U10.4 (I4)
- new net MAIN_OUT_OD: J9.15 (Pin_15), U10.13 (O4)
- new net PRECHARGE_OUT: U10.3 (I3)
- new net PRECHARGE_OUT_OD: J9.13 (Pin_13), U10.14 (O3)
- new net PUMP_OUT: U10.1 (I1)
- new net PUMP_OUT_OD: J9.9 (Pin_9), U10.16 (O1)
- new net X_OUT_OD: J9.17 (Pin_17), U10.12 (O5), U10.5 (I5)
- no-connect marks 1 -> 5
Other:
- note added: "CAN TRX"
- note added: "Current Sensing"
- note added: "DRIVER"
- note added: "Input/Output"
- note added: "Power"
- note added: "Resolver"
- note added: "Unconnected!!!"
- note added: "Virtual ground"
- note added: "Zrob Cos z VBUSEM !!!!"
- note removed: "Można zmienić na ten z oryginalnej płytki"
- moved on the sheet: C1, C10, C2, C21, C22, C23, C27, C3, C33, C4, C5, C6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

Commit message: Added High current OD and comparators
Parts:
- added D8: 1N4148, Diode_SMD:D_SOD-323, symbol MEMS_Discrete_Semiconductors:D_1N4148WS-SOD323
- added JP1, JP2: ~, MEMS_Passive:R_0805_2012Metric_Jumper, symbol MEMS_Passive:SolderableJumper
- added Q4: ST3422A, Package_TO_SOT_SMD:SOT-23-3, symbol Device:Q_NMOS_GSD
- added R46, R47, R48, R49: ~, Resistor_SMD:R_0603_1608Metric, symbol Device:R
- added R50: 10k, Resistor_SMD:R_0603_1608Metric_Pad0.98x0.95mm_HandSolder, symbol Device:R
- added U11, U12: LM393, symbol Comparator:LM393
Connections:
- net +3V3: now also R50.1
- net +5V: now also R46.1, R48.1, U11.8 (V+), U12.8 (V+)
- net FAULT_DRV: now also U11.1, U11.7, U12.1, U12.7
- net GND: now also D8.2 (A), Q4.2 (S), R47.2, R49.2, U11.4 (V-), U12.4 (V-)
- net MAIN_OUT: now also U10.6 (I6), R50.2; no longer U10.4 (I4)
- net MAIN_OUT_OD: now also D8.1 (K), Q4.3 (D); no longer U10.13 (O4)
- net PWM_DRIVER/DRIVER_OUTPUT_ENABLE: now also U4.2, U4.6
- net SWCLK: now also J1.3 (Pin_3), JP1.1; no longer J9.14 (Pin_14)
- net SWDIO: now also J1.2 (Pin_2), JP2.1; no longer J9.12 (Pin_12)
- net X_OUT_OD: no longer U10.5 (I5)
- net CURRENT_B_RAW: now reaches J7.4 (Pin_4), R25.1
- net CURRENT_B_RAW: now also U11.3 (+), U12.2 (-)
- net CURRENT_A_RAW: now reaches J7.2 (Pin_2), R27.1
- net CURRENT_A_RAW: now also U11.6 (-), U12.5 (+)
- net at U10.11 (O6): now also Q4.1 (G)
- new net: J9.14 (Pin_14), JP1.2
- new net: J9.12 (Pin_12), JP2.2
- new net NEG_CURRENT_SETPOINT: R46.2, R47.1, U11.5 (+), U12.3 (+)
- new net POS_CURRENT_SETPOINT: R48.2, R49.1, U11.2 (-), U12.6 (-)
- new net X_OUT: U10.5 (I5)
- no-connect marks 5 -> 3
Other:
- moved on the sheet: C10, C9, D5, H1, H2, H3, H4, J1, J5, J7, R18, R23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
