File: STM32Inverter.kicad_sch (KiCad schematic)
At the start: 94 parts, among them J1 STLINK, J2 RESOLVER, J3 MAIN POWER, J4 Power, J5 UART, J7 CURRENT SENSE, J8 DRIVER BOARD, J9 INTERFACE, Q4 ST3422A, U1 STM32F303VCTx, U10 ULN2002, U11 LM393, U12 LM393, U4 74HCT00, U7 MCP2551-I-SN, Y3 CSTNE8M00GH5C000R0

Commit message: Added libraries, NTC
Parts:
- removed J2: RESOLVER, Connector_IDC:IDC-Header_2x06_P2.54mm_Vertical, symbol Connector_Generic:Conn_02x06_Odd_Even
- removed J7: CURRENT SENSE, Connector_JST:JST_PH_B4B-PH-K_1x04_P2.00mm_Vertical, symbol Connector:Conn_01x04_Pin
- removed J8: DRIVER BOARD, Connector_IDC:IDC-Header_2x10_P2.54mm_Vertical, symbol Connector_Generic:Conn_02x10_Odd_Even
- removed J9: INTERFACE, Connector_IDC:IDC-Header_2x10_P2.54mm_Vertical, symbol Connector_Generic:Conn_02x10_Odd_Even
- added J2: CURRENT SENSE, DF51K4P2DS805, symbol DF51K-4P-2DS_805_:DF51K-4P-2DS_805_
- added J6: INTERFACE, DF51-20:DF51K20DP2DS805, symbol DF51K-20DP-2DS_805_:DF51K-20DP-2DS_805_
- added J8: 501571-2007, picoclasp:5015712007, symbol 501571-2007:501571-2007
- added J9: RESOLVER, DF51-20:DF51K20DP2DS805, symbol DF51K-20DP-2DS_805_:DF51K-20DP-2DS_805_
- added R51: 10k, Resistor_SMD:R_0603_1608Metric_Pad0.98x0.95mm_HandSolder, symbol Device:R
- added TH1: Thermistor_NTC, Resistor_SMD:R_0805_2012Metric_Pad1.20x1.40mm_HandSolder, symbol Device:Thermistor_NTC
- U11, U12: footprint (none) -> Package_SO:SOP-8_3.9x4.9mm_P1.27mm; LCSC (none) -> C5252905
Connections:
- net +12_EXT: now also J6.1, J6.3
- net +3V3: now also R51.1
- net +5V: now also J2.1, J8.17, J8.19
- net +5VA: now also J8.2
- net CAN_H: now also J6.2
- net CAN_L: now also J6.4
- net COS_H: now also J9.1
- net COS_L: now also J9.3
- net CURRENT_A_RAW: now also J2.2
- net CURRENT_B_RAW: now also J2.4
- net EXC: now also J9.9
- net FAN_OUT_OD: now also J6.11
- net FAULT_DRV: now also J8.4
- net GND: now also J2.3, J6.10, J6.5, J6.7, J8.7, J8.9, J9.12, J9.2, TH1.2
- net MAIN_OUT_OD: now also J6.15
- net PRECHARGE_OUT_OD: now also J6.13
- net PUMP_OUT_OD: now also J6.9
- net SIN_H: now also J9.5
- net SIN_L: now also J9.7
- net T1_DRV: now also J8.10
- net T2_DRV: now also J8.12
- net T3_DRV: now also J8.14
- net TG1: now also J9.4
- net TG2: now also J9.8
- net TH1: now also J9.6
- net TH2: now also J9.10
- net U_HIGH: now also J8.1
- net U_LOW: now also J8.11
- net V_HIGH: now also J8.5
- net V_LOW: now also J8.15
- net W_HIGH: now also J8.3
- net W_LOW: now also J8.13
- net X_OUT_OD: now also J6.17
- net ~{EXC}: now also J9.11
- net at R44.1: now also J6.19
- net at R42.1: now also J6.20
- net at TP8.1: now also J8.6
- net at F3.2: now also J6.16
- net at TP6.1: now also J8.18
- net at JP1.2: now also J6.14
- net at R35.1: now also J8.8
- net at R33.1: now also J6.8
- net at JP2.2: now also J6.12
- net at TP7.1: now also J8.16
- net at R38.1: now also J6.6
- net at R40.1: now also J6.18
- net at TP5.1: now also J8.20
- new net TEMP_INTERNAL: R51.2, TH1.1
Other:
- moved on the sheet: C17, C29, D8, D9A, D9B, D9C, D9D, F3, JP1, JP2, Q4, R31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

Commit message: Final version before layout
Parts:
- removed J3: MAIN POWER, Connector_JST:JST_XH_B2B-XH-AM_1x02_P2.50mm_Vertical, symbol Connector:Conn_01x02_Pin
- removed J4: Power, Connector_PinHeader_2.54mm:PinHeader_1x06_P2.54mm_Vertical, symbol Connector:Conn_01x06_Pin
- added D11, D12: BZT52C3V6, Diode_SMD:D_SOD-123, symbol Device:D_Zener
- added J7: POWER, DF51K8DP2DS805, symbol DF51K-8DP-2DS_805_:DF51K-8DP-2DS_805_
- added R52, R53: 10k, Resistor_SMD:R_0603_1608Metric_Pad0.98x0.95mm_HandSolder, symbol Device:R
- R50: value 10k -> 2.2k
Connections:
- net TG1 is gone; now on net GND: J9.4
- net TG2 is gone; now on net GND: J9.8
- net +12_UNSTABILIZED: now also J7.6, J7.8
- net +3V3: now also R52.1, R53.1
- net +5VA: now also J7.5
- net GND: now also J8.MP1, J8.MP2, D11.2 (A), D12.2 (A), J7.2, J7.4
- net MAIN_OUT: now also U10.5 (I5); no longer U10.6 (I6)
- net TH1: now also D12.1 (K), R52.2
- net TH2: now also D11.1 (K), R53.2
- net X_OUT: now also U10.4 (I4); no longer U10.5 (I5)
- net X_OUT_OD: now also U10.13 (O4); no longer U10.12 (O5)
- net at F2.2: now also J7.1
- net at F4.2: now also J7.7
- net at F1.2: now also J7.3
- net at Q4.1 (G): now also U10.12 (O5); no longer U10.11 (O6)
- no-connect marks 3 -> 5
Other:
- note added: "Dobrać bezpieczniki"
- note added: "TG1"
- note added: "TG2"
- moved on the sheet: C1, C2, C21, C22, C23, C3, C33, C4, C5, C6, C7, D4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

Commit message: Resolver layout
Parts:
- J2: footprint DF51K4P2DS805 -> DF51-4:DF51K4P2DS805
- J7: footprint DF51K8DP2DS805 -> DF51-8:DF51K8DP2DS805
Changed lines of the file:
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@@
       (effects (font (size 1.27 1.27)))
     )
-    (property "Footprint" "DF51K4P2DS805" (at 20.32 215.57 0)
+    (property "Footprint" "DF51-4:DF51K4P2DS805" (at 20.32 215.57 0)
       (effects (font (size 1.27 1.27)) (justify left top) hide)
     )
@@
       (effects (font (size 1.27 1.27)))
     )
-    (property "Footprint" "DF51K8DP2DS805" (at 63.5 395.91 0)
+    (property "Footprint" "DF51-8:DF51K8DP2DS805" (at 63.5 395.91 0)
       (effects (font (size 1.27 1.27)) (justify left top) hide)
     )

Commit message: Layout mostly done
Parts:
- U11, U12: footprint Package_SO:SOP-8_3.9x4.9mm_P1.27mm -> Package_SO:SO-8_3.9x4.9mm_P1.27mm
Connections:
- net +12_EXT: now also J6.17, J6.19; no longer J6.1, J6.3
- net FAN_OUT_OD: now also J6.5; no longer J6.11
- net GND: now also J6.13, J6.15; no longer J6.5, J6.7
- net MAIN_OUT_OD: now also J6.9; no longer J6.15
- net PRECHARGE_OUT_OD: now also J6.7; no longer J6.13
- net PUMP_OUT_OD: now also J6.3; no longer J6.9
- net X_OUT_OD: now also J6.11; no longer J6.17
- net at R44.1: now also J6.1; no longer J6.19
Other:
- moved on the sheet: C17, C29, D8, D9A, D9B, D9C, D9D, F3, J6, JP1, JP2, Q4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

Commit message: Traces almost done
Connections:
- net 2.5V: now also U1.16 (PC1), U1.18 (PC3)
- net AUX_IN: now also D9.4 (K3); no longer D9.6 (K5)
- net CURRENT_A: now also U1.15 (PC0)
- net CURRENT_B: now also U1.17 (PC2)
- net KEY_IN: now also D9.6 (K5); no longer D9.4 (K3)
- net T1_DRV: now also U1.27 (PF4)
- net T2_DRV: now also U1.26 (PA3)
- net T3_DRV: now also U1.19 (PF2)
- net TH1: now also U1.39 (PE8)
- net TH2: now also U1.45 (PE14)
Other:
- note added: "CHECK STLINK!!!!"
- note added: "Check if you can swap ADC +- pins"

Commit message: Board done
Connections:
- net +12_EXT_ADC: now also U1.56 (PD9)
- net ACC_INPUT_A_3V3: now also U1.54 (PB15)
- net ACC_INPUT_B_3V3: now also U1.53 (PB14)
- net AUX_IN: now also U1.58 (PD11)
- net BRK_IN: now also U1.60 (PD13)
- net DOS: now also U1.52 (PB13)
- net FAN_OUT: now also U1.79 (PC11)
- net FAULT_RST: now also U1.5 (PE6)
- net FAULT_SR_3V3: now also U1.4 (PE5)
- net KEY_IN: now also U1.59 (PD12)
- net LOT: now also U1.51 (PB12)
- net MAIN_OUT: now also U1.81 (PD0)
- net PRECHARGE_OUT: now also U1.78 (PC10)
- net PUMP_OUT: now also U1.80 (PC12)
- net TEMP_INTERNAL: now also U1.57 (PD10)
- net VBUS_DRV: now also U1.55 (PD8)
- net X_OUT: now also U1.77 (PA15)
Changed lines of the file:
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@@
+    (stroke (width 0) (type default))
+  )
+  (wire (pts (xy 218.44 242.57) (xy 233.68 242.57))
+    (stroke (width 0) (type default))
+  )
+  (wire (pts (xy 218.44 250.19) (xy 233.68 250.19))
     (stroke (width 0) (type default))
   )
@@
     (stroke (width 0) (type default))
   )
+  (wire (pts (xy 294.64 217.17) (xy 274.32 217.17))
+    (stroke (width 0) (type default))
+  )
   (wire (pts (xy 35.56 170.18) (xy 35.56 172.72))
     (stroke (width 0) (type default))
@@
     (stroke (width 0) (type default))
   )
+  (wire (pts (xy 219.71 189.23) (xy 233.68 189.23))
+    (stroke (width 0) (type default))
+  )
   (wire (pts (xy 36.83 26.67) (xy 36.83 59.69))
     (stroke (width 0) (type default))
@@
     (stroke (width 0) (type default))
   )
+  (wire (pts (xy 297.18 250.19) (xy 274.32 250.19))
+    (stroke (width 0) (type default))
+  )
   (wire (pts (xy 448.31 34.29) (xy 459.74 34.29))
     (stroke (width 0) (type default))
@@
     (stroke (width 0) (type default))
   )
+  (wire (pts (xy 222.25 217.17) (xy 233.68 217.17))
+    (stroke (width 0) (type default))
+  )
   (wire (pts (xy 262.89 81.28) (xy 262.89 55.88))
     (stroke (width 0) (type default))
@@
     (stroke (width 0) (type default))
   )
+  (wire (pts (xy 218.44 240.03) (xy 233.68 240.03))
+    (stroke (width 0) (type default))
+  )
   (wire (pts (xy 36.83 358.14) (xy 45.72 358.14))
     (stroke (width 0) (type default))
@@
     (stroke (width 0) (type default))
   )
+  (wire (pts (xy 283.21 212.09) (xy 274.32 212.09))
+    (stroke (width 0) (type default))
+  )
   (wire (pts (xy 96.52 266.7) (xy 100.33 266.7))
     (stroke (width 0) (type default))
@@
     (stroke (width 0) (type default))
   )
+  (wire (pts (xy 292.1 176.53) (xy 274.32 176.53))
+    (stroke (width 0) (type default))
+  )
   (wire (pts (xy 509.27 184.15) (xy 509.27 185.42))
     (stroke (width 0) (type default))
@@
     (stroke (width 0) (type default))
   )
+  (wire (pts (xy 283.21 214.63) (xy 274.32 214.63))
+    (stroke (width 0) (type default))
+  )
   (wire (pts (xy 281.94 153.67) (xy 274.32 153.67))
     (stroke (width 0) (type default))
@@
     (stroke (width 0) (type default))
   )
+  (wire (pts (xy 297.18 255.27) (xy 274.32 255.27))
+    (stroke (width 0) (type default))
+  )
   (wire (pts (xy 518.16 132.08) (xy 511.81 132.08))
     (stroke (width 0) (type default))
@@
     (stroke (width 0) (type default))
   )
+  (wire (pts (xy 218.44 247.65) (xy 233.68 247.65))
+    (stroke (width 0) (type default))
+  )
   (wire (pts (xy 224.79 158.75) (xy 233.68 158.75))
     (stroke (width 0) (type default))
@@
     (stroke (width 0) (type default))
   )
+  (wire (pts (xy 294.64 219.71) (xy 274.32 219.71))
+    (stroke (width 0) (type default))
+  )
   (wire (pts (xy 255.27 330.2) (xy 255.27 327.66))
     (stroke (width 0) (type default))
@@
     (stroke (width 0) (type default))
   )
+  (wire (pts (xy 218.44 237.49) (xy 233.68 237.49))
+    (stroke (width 0) (type default))
+  )
   (wire (pts (xy 133.35 46.99) (xy 133.35 59.69))
     (stroke (width 0) (type default))
@@
     (stroke (width 0) (type default))
   )
+  (wire (pts (xy 297.18 252.73) (xy 274.32 252.73))
+    (stroke (width 0) (type default))
+  )
   (wire (pts (xy 49.53 68.58) (xy 44.45 68.58))
     (stroke (width 0) (type default))
@@
     (stroke (width 0) (type default))
   )
+  (wire (pts (xy 218.44 245.11) (xy 233.68 245.11))
+    (stroke (width 0) (type default))
+  )
   (wire (pts (xy 45.72 345.44) (xy 45.72 347.98))
     (stroke (width 0) (type default))
@@
   )
   (wire (pts (xy 518.16 137.16) (xy 511.81 137.16))
+    (stroke (width 0) (type default))
+  )
+  (wire (pts (xy 219.71 186.69) (xy 233.68 186.69))
     (stroke (width 0) (type default))
   )
@@
     (effects (font (size 1.27 1.27)) (justify left bottom))
   )
-  (label "+12_EXT_ADC" (at 364.49 260.35 0) (fields_autoplaced)
+  (label "+12_EXT_ADC" (at 218.44 240.03 0) (fields_autoplaced)
     (effects (font (size 1.27 1.27)) (justify left bottom))
   )
@@
     (effects (font (size 1.27 1.27)) (justify right bottom))
   )
-  (label "DOS" (at 358.14 260.35 0) (fields_autoplaced)
-    (effects (font (size 1.27 1.27)) (justify left bottom))
+  (label "DOS" (at 283.21 214.63 180) (fields_autoplaced)
+    (effects (font (size 1.27 1.27)) (justify right bottom))
   )
   (label "CURRENT_B" (at 102.87 137.16 0) (fields_autoplaced)
@@
     (effects (font (size 1.27 1.27)) (justify left bottom))
   )
+  (label "PUMP_OUT" (at 297.18 255.27 180) (fields_autoplaced)
+    (effects (font (size 1.27 1.27)) (justify right bottom))
+  )
   (label "CURRENT_A" (at 297.18 224.79 180) (fields_autoplaced)
     (effects (font (size 1.27 1.27)) (justify right bottom))
@@
     (effects (font (size 1.27 1.27)) (justify left bottom))
   )
-  (label "LOT" (at 358.14 262.89 0) (fields_autoplaced)
-    (effects (font (size 1.27 1.27)) (justify left bottom))
+  (label "LOT" (at 283.21 212.09 180) (fields_autoplaced)
+    (effects (font (size 1.27 1.27)) (justify right bottom))
   )
   (label "PWM_CH2N" (at 394.97 35.56 0) (fields_autoplaced)
@@
     (effects (font (size 1.27 1.27)) (justify right bottom))
   )
-  (label "VBUS_DRV" (at 359.41 275.59 180) (fields_autoplaced)
-    (effects (font (size 1.27 1.27)) (justify right bottom))
+  (label "VBUS_DRV" (at 218.44 237.49 0) (fields_autoplaced)
+    (effects (font (size 1.27 1.27)) (justify left bottom))
   )
   (label "FAULT_RST" (at 422.91 95.25 0) (fields_autoplaced)
@@
     (effects (font (size 1.27 1.27)) (justify right bottom))
   )
-  (label "TEMP_INTERNAL" (at 365.76 280.67 0) (fields_autoplaced)
+  (label "TEMP_INTERNAL" (at 218.44 242.57 0) (fields_autoplaced)
     (effects (font (size 1.27 1.27)) (justify left bottom))
   )
@@
     (effects (font (size 1.27 1.27)) (justify left bottom))
   )
-  (label "AUX_IN" (at 367.03 276.86 0) (fields_autoplaced)
+  (label "AUX_IN" (at 218.44 245.11 0) (fields_autoplaced)
     (effects (font (size 1.27 1.27)) (justify left bottom))
   )
@@
     (effects (font (size 1.27 1.27)) (justify right bottom))
   )
-  (label "FAULT_RST" (at 341.63 262.89 0) (fields_autoplaced)
+  (label "FAULT_RST" (at 219.71 189.23 0) (fields_autoplaced)
     (effects (font (size 1.27 1.27)) (justify left bottom))
   )
@@
     (effects (font (size 1.27 1.27)) (justify left bottom))
   )
-  (label "FAN_OUT" (at 374.65 254 0) (fields_autoplaced)
-    (effects (font (size 1.27 1.27)) (justify left bottom))
+  (label "FAN_OUT" (at 297.18 252.73 180) (fields_autoplaced)
+    (effects (font (size 1.27 1.27)) (justify right bottom))
   )
   (label "T2_DRV" (at 281.94 146.05 0) (fields_autoplaced)
@@
     (effects (font (size 1.27 1.27)) (justify left bottom))
   )
-  (label "BRK_IN" (at 377.19 273.05 180) (fields_autoplaced)
-    (effects (font (size 1.27 1.27)) (justify right bottom))
+  (label "BRK_IN" (at 218.44 250.19 0) (fields_autoplaced)
+    (effects (font (size 1.27 1.27)) (justify left bottom))
   )
   (label "BRK_IN" (at 147.32 68.58 180) (fields_autoplaced)
@@
     (effects (font (size 1.27 1.27)) (justify left bottom))
   )
-  (label "ACC_INPUT_B_3V3" (at 375.92 270.51 180) (fields_autoplaced)
+  (label "ACC_INPUT_B_3V3" (at 294.64 217.17 180) (fields_autoplaced)
     (effects (font (size 1.27 1.27)) (justify right bottom))
   )
@@
     (effects (font (size 1.27 1.27)) (justify left bottom))
   )
-  (label "PRECHARGE_OUT" (at 374.65 256.54 0) (fields_autoplaced)
-    (effects (font (size 1.27 1.27)) (justify left bottom))
+  (label "PRECHARGE_OUT" (at 297.18 250.19 180) (fields_autoplaced)
+    (effects (font (size 1.27 1.27)) (justify right bottom))
   )
   (label "2.5V" (at 288.29 227.33 0) (fields_autoplaced)
@@
     (effects (font (size 1.27 1.27)) (justify right bottom))
   )
-  (label "PUMP_OUT" (at 374.65 251.46 0) (fields_autoplaced)
-    (effects (font (size 1.27 1.27)) (justify left bottom))
-  )
   (label "~{EXC}" (at 444.5 144.78 0) (fields_autoplaced)
     (effects (font (size 1.27 1.27)) (justify left bottom))
   )
-  (label "KEY_IN" (at 344.17 273.05 180) (fields_autoplaced)
-    (effects (font (size 1.27 1.27)) (justify right bottom))
+  (label "KEY_IN" (at 218.44 247.65 0) (fields_autoplaced)
+    (effects (font (size 1.27 1.27)) (justify left bottom))
   )
   (label "PWM_CH2" (at 394.97 33.02 0) (fields_autoplaced)
@@
     (effects (font (size 1.27 1.27)) (justify right bottom))
   )
-  (label "X_OUT" (at 335.28 278.13 0) (fields_autoplaced)
-    (effects (font (size 1.27 1.27)) (justify left bottom))
+  (label "X_OUT" (at 292.1 176.53 180) (fields_autoplaced)
+    (effects (font (size 1.27 1.27)) (justify right bottom))
   )
   (label "CURRENT_A_RAW" (at 77.47 119.38 90) (fields_autoplaced)
@@
     (effects (font (size 1.27 1.27)) (justify right bottom))
   )
-  (label "FAULT_SR_3V3" (at 341.63 260.35 0) (fields_autoplaced)
+  (label "FAULT_SR_3V3" (at 219.71 186.69 0) (fields_autoplaced)
     (effects (font (size 1.27 1.27)) (justify left bottom))
   )
@@
     (effects (font (size 1.27 1.27)) (justify left bottom))
   )
-  (label "ACC_INPUT_A_3V3" (at 353.06 270.51 180) (fields_autoplaced)
+  (label "ACC_INPUT_A_3V3" (at 294.64 219.71 180) (fields_autoplaced)
     (effects (font (size 1.27 1.27)) (justify right bottom))
   )
@@
     (effects (font (size 1.27 1.27)) (justify left bottom))
   )
-  (label "MAIN_OUT" (at 377.19 265.43 0) (fields_autoplaced)
-    (effects (font (size 1.27 1.27)) (justify left bottom))
-  )
+  (label "MAIN_OUT" (at 222.25 217.17 0) (fields_autoplaced)
+    (effects (font (size 1.27 1.27)) (justify left bottom))
+  )

Commit message: Board enven more done
Connections:
- net LED_PIN: now also U1.73 (PF6)
Changed lines of the file:
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@@
+    (stroke (width 0) (type default))
+  )
+  (wire (pts (xy 224.79 163.83) (xy 233.68 163.83))
     (stroke (width 0) (type default))
   )
@@
     (effects (font (size 1.27 1.27)) (justify left bottom))
   )
+  (label "LED_PIN" (at 224.79 163.83 0) (fields_autoplaced)
+    (effects (font (size 1.27 1.27)) (justify left bottom))
+  )

Commit message: Awaiting review
Other:
- note added: "Driver"
- note removed: "Add proper jellybeans"
- note removed: "DIFFERENTIAL"
- note removed: "DRIVER"
- note removed: "Dobrać bezpieczniki"
- note removed: "PINS TO ARRANGE!!!"
- note removed: "Unconnected!!!"
- moved on the sheet: C27, R21, R22, U7
