File: STM32Inverter.kicad_pcb (KiCad board)
At the start: 4 copper layers, 100 x 100 mm, 151 parts, among them J1 STLINK, J2 CURRENT SENSE, J5 UART, J6 INTERFACE, J7 POWER, J8 501571-2007, J9 RESOLVER, Q1 BCX54, Q2 BCX55, Q4 ST3422A, Q5 BCX54, Q6 BCX55, U1 STM32F303VCTx, U10 ULN2002, U11 LM393, U12 LM393, U2 LM358, U3 AD2S1205, U4 74HCT00, U5 74HCT04, U6 74HCT08, U7 MCP2551-I-SN, U8 74HCT08, U9 74HCT08, Y2 CSTNE8M00GH5C000R0, Y3 CSTNE8M00GH5C000R0

Commit message: Board done
Parts:
- moved R51 2.00 mm to (69.5, 30.8)
- moved TH1 2.00 mm to (65.2, 30.8)
- moved C1 0.17 mm to (53.2, 41.8)
Connections:
- U1 pad 4: unconnected-(U1-PE5-Pad4) -> /FAULT_SR_3V3
- U1 pad 5: unconnected-(U1-PE6-Pad5) -> /FAULT_RST
- U1 pad 51: unconnected-(U1-PB12-Pad51) -> /LOT
- U1 pad 52: unconnected-(U1-PB13-Pad52) -> /DOS
- U1 pad 53: unconnected-(U1-PB14-Pad53) -> /ACC_INPUT_B_3V3
- U1 pad 54: unconnected-(U1-PB15-Pad54) -> /ACC_INPUT_A_3V3
- U1 pad 55: unconnected-(U1-PD8-Pad55) -> /VBUS_DRV
- U1 pad 56: unconnected-(U1-PD9-Pad56) -> /+12_EXT_ADC
- U1 pad 57: unconnected-(U1-PD10-Pad57) -> /TEMP_INTERNAL
- U1 pad 58: unconnected-(U1-PD11-Pad58) -> /AUX_IN
- U1 pad 59: unconnected-(U1-PD12-Pad59) -> /KEY_IN
- U1 pad 60: unconnected-(U1-PD13-Pad60) -> /BRK_IN
- U1 pad 77: unconnected-(U1-PA15-Pad77) -> /X_OUT
- U1 pad 78: unconnected-(U1-PC10-Pad78) -> /PRECHARGE_OUT
- U1 pad 79: unconnected-(U1-PC11-Pad79) -> /FAN_OUT
- U1 pad 80: unconnected-(U1-PC12-Pad80) -> /PUMP_OUT
- U1 pad 81: unconnected-(U1-PD0-Pad81) -> /MAIN_OUT
Routing:
- net /VBUS_DRV: track 1.85 -> 85.0 mm, vias 0 -> 2
- net /+12_EXT_ADC: track 0.00 -> 45.0 mm, vias 0 -> 3
- net /FAULT_RST: track 1.27 -> 45.6 mm, vias 0 -> 4
- net /PRECHARGE_OUT: track 0.00 -> 42.2 mm, vias 0 -> 3
- net /FAULT_SR_3V3: track 1.95 -> 44.0 mm, vias 0 -> 2
- net /X_OUT: track 0.00 -> 41.8 mm, vias 0 -> 3
- net /PUMP_OUT: track 0.00 -> 40.5 mm, vias 0 -> 3
- net /FAN_OUT: track 0.00 -> 38.1 mm, vias 0 -> 3
- net /DOS: track 2.14 -> 37.5 mm, vias 1 -> 2
- net /LOT: track 1.73 -> 34.3 mm, vias 1 -> 2
- net /TEMP_INTERNAL: track 0.00 -> 32.0 mm, vias 0 -> 2
- net /AUX_IN: track 21.7 -> 50.3 mm, vias 0 -> 2
- net /MAIN_OUT: track 19.0 -> 47.3 mm, vias 0 -> 3
- net /KEY_IN: track 15.3 -> 39.2 mm, vias 0 -> 2
- net /BRK_IN: track 12.7 -> 29.2 mm, vias 0 -> 2
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